Commit message: ROS2 Galactic ver. Nav2 패키지 파라미터 변경. 로봇 URDF 수정. 테스트 SLAM, NAV2 진행 완료.

File: src/STELLA_REMOTE_PC_ROS2_N2/stella_description/urdf/stella.urdf (robot description, URDF)
Before this commit: robot stella, 4 links, 3 joints
Links:
- link base_link: geometry collision box size=0.240 0.250 0.610; visual mesh filename=package://stella_description/meshes/bases/STELLA-N2.stl scale=0.001 0.001 0.001
Joints:
- joint imu_joint: origin xyz=-0.06 0.0 0.063 rpy=0.0 0.0 0.0 -> xyz=-0.06 0.0 0.610 rpy=0.0 0.0 0.0
- joint scan_joint: origin xyz=0.06 0.0 0.159 rpy=0.0 0.0 0.0 -> xyz=0.06 0.0 0.710 rpy=0.0 0.0 0.0

Commit message: 릴레이 노드 테스트용 코드 수정

File: src/STELLA_REMOTE_PC_ROS2_N2/stella_description/urdf/stella.urdf (robot description, URDF)
Before this commit: robot stella, 4 links, 3 joints
Links:
- link base_link: geometry collision box size=0.17 0.207 0.164; visual mesh filename=package://stella_description/meshes/bases/STELLA-N2.stl scale=0.001 0.001 0.001
Joints:
- joint imu_joint: origin xyz=-0.06 0.0 0.610 rpy=0.0 0.0 0.0 -> xyz=-0.06 0.0 0.063 rpy=0.0 0.0 0.0
- joint scan_joint: origin xyz=0.06 0.0 0.710 rpy=0.0 0.0 0.0 -> xyz=0.06 0.0 0.159 rpy=0.0 0.0 0.0
